File: ahoy_pcb/ahoy_pcb.kicad_pcb (KiCad board)
At the start: 2 copper layers, 123.8 x 95.2 mm, 107 parts, among them J1 TYPE-C-31-M12_13, P1 TC2030-AVR, SW1 SW_Push, SW2 Rotary_Encoder_Switch_Chassis, U1 ATmega32U4-A, U2 USBLC6-2SC6, Y1 16MHz

Commit message: More updates
Parts:
- removed C10, C11, C12, C13, C14, C15, C8, C9: 10uF, Capacitor_SMD:C_0805_2012Metric
- removed LED1, LED2, LED3, LED4, LED5, LED6, LED7, LED8: WS2812B, Acheron Components:LED_WS2812B-Mini_3.5x3.5mm
- added C16: 0.1uF, Capacitor_SMD:C_0805_2012Metric, B.Cu at (60.8, 79.8)
- added J2: Conn_01x03_Female, Acheron Connectors:PinHeader_1x3_staggered_P2.54mm_Vertical, F.Cu at (66.4, 138.3)
- moved P1 46.4 mm to (75.7, 69.6)
- moved SW1 41.5 mm to (90.6, 73.0), turned to 0 degrees
- moved R10 23.2 mm to (65.5, 141.2)
- moved C6 21.3 mm to (74.4, 83.5), turned to 0 degrees
- moved C4 18.6 mm to (56.1, 91.0)
- moved C7 15.5 mm to (60.8, 75.9), turned to 180 degrees
- moved F1 13.4 mm to (61.3, 69.8)
- moved R2 9.08 mm to (67.4, 70.4)
- moved R1 9.08 mm to (65.3, 70.4)
- moved C3 2.85 mm to (68.2, 75.4)
- moved R3 2.50 mm to (71.4, 74.7), turned to 0 degrees
- moved D31 0.51 mm to (66.7, 132.8)
- moved D32 0.51 mm to (66.7, 128.3)
- moved D33 0.51 mm to (66.7, 123.7)
- moved R7 0.51 mm to (62.6, 133.2)
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Connections:
- net Net-(R1-Pad2) renamed /PostRD-
- net Net-(R2-Pad1) renamed /PostRD+
- C2 pad 1: GND -> Net-(C2-Pad1)
- C2 pad 2: Net-(C2-Pad2) -> GND
- U1 pad 16: Net-(C2-Pad2) -> Net-(C2-Pad1)
- Y1 pad 1: Net-(C2-Pad2) -> Net-(C1-Pad2)
- Y1 pad 3: Net-(C1-Pad2) -> Net-(C2-Pad1)
Routing:
- net +5V: track 627.2 -> 158.7 mm, vias 13 -> 7
- net GND: track 58.0 -> 307.0 mm, vias 17 -> 11
- net Net-(LED4-Pad2): track 86.9 -> 0.00 mm
- net Net-(LED5-Pad2): track 61.4 -> 0.00 mm
- net Net-(LED1-Pad2): track 57.3 -> 0.00 mm
- net Col2: track 165.7 -> 114.6 mm
- net Net-(LED3-Pad2): track 50.3 -> 0.00 mm, vias 2 -> 0
- net Col4: track 187.4 -> 138.1 mm, vias 1 -> 3
- net Net-(LED6-Pad2): track 48.6 -> 0.00 mm
- net Col3: track 166.4 -> 118.0 mm, vias 1 -> 3
- net Row1: track 212.7 -> 164.6 mm, vias 6 -> 2
- net Row2: track 163.5 -> 115.9 mm
- net Col5: track 208.3 -> 160.8 mm, vias 1 -> 3
- net Net-(LED7-Pad2): track 40.4 -> 0.00 mm
- net Net-(LED2-Pad2): track 37.2 -> 0.00 mm
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