File: ahoy_pcb/ahoy_pcb.kicad_sch (KiCad schematic)
At the start: 107 parts, among them J1 TYPE-C-31-M12_13, P1 TC2030-AVR, SW1 SW_Push, SW2 Rotary_Encoder_Switch_Chassis, U1 ATmega32U4-A, U2 USBLC6-2SC6, Y1 16MHz

Commit message: More updates
Parts:
- removed C10, C11, C12, C13, C14, C15, C8, C9: 10uF, Capacitor_SMD:C_0805_2012Metric, symbol Device:C_Small
- removed LED1, LED2, LED3, LED4, LED5, LED6, LED7, LED8: WS2812B, Acheron Components:LED_WS2812B-Mini_3.5x3.5mm, symbol ws2812b:WS2812B
- added C16: 0.1uF, Capacitor_SMD:C_0805_2012Metric, symbol Device:C_Small
- added J2: Conn_01x03_Female, Acheron Connectors:PinHeader_1x3_staggered_P2.54mm_Vertical, symbol Connector:Conn_01x03_Female
Connections:
- net +5V: now also C16.1, J2.3 (Pin_3)
- net GND: now also C2.2, C16.2, J2.1 (Pin_1); no longer C2.1
- net at C1.2, U1.17 (XTAL1): now also Y1.1; no longer Y1.3
- net PostRD-: now reaches R1.2, U1.3 (D-)
- net at R10.1: now also J2.2 (Pin_2)
- net PostRD+: now reaches R2.1, U1.4 (D+)
- new net: C2.1, U1.16 (XTAL2), Y1.3
- no-connect marks 10 -> 9
Other:
- note added: "AVR ISP Breakout"
- note added: "ESD Protection"
- note added: "RGB Breakout"
- note added: "Rotary Encoder"
- moved on the sheet: C1, C2, D1, D10, D11, D12, D13, D14, D15, D16, D17, D18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
